File: Kicad/hapsole.kicad_sch (KiCad schematic)
At the start: 31 parts, among them J1 USB_C_Receptacle_USB2.0_16P, Q1 PMOS, U1 DA7280-00V42, U2 DA7280-00V42, U3 nRF52840, U4 LSM6DS3TR-C, U5 BQ25100YFPR, U6 TLV73333PDBV, Y1 32.768Khz

Commit message: Added i2c Pins
Parts:
- added C6, C7, C8, C9: C, symbol Device:C
Connections:
- net 6D_INT1: now also U3.T2 (TRACEDATA2/P0.11)
- net 6D_PWR: now also U3.P2 (P1.08)
- net GND: now also C6.1, C7.1, C8.2, C9.2
- net INTERNAL_I2C_SCL: now also U3.H2 (P0.27)
- net INTERNAL_I2C_SDA: now also U3.M2 (TRACECLK/P0.07)
- net at U3.F2 (XL2/P0.01), Y1.1: now also C7.2
- net at U3.D2 (XL1/P0.00), Y1.2: now also C6.2
- net at U3.AC5 (DECUSB): now also C9.1
- net at U3.C1 (DEC1): now also C8.1
