File: Kicad/hapsole.kicad_pcb (KiCad board)
At the start: 4 copper layers, 33.5 x 22.6 mm, 64 parts, among them J1 2171790001, J2 Conn_01x02_Socket, J3 Conn_01x02_Socket, Q1 PMOS, U1 DA7281-00FV2, U2 DA7281-00FV2, U3 nRF52840, U4 LSM6DS3TR-C, U5 BQ25100YFPR, U6 TLV73333PDBV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

Commit message: finished arrangement of all components
Parts:
- U7: footprint Package_SO:SOIC-8_5.3x5.3mm_P1.27mm -> Hapsole_Custom:Untitled; moved to B.Cu
- U8: moved to B.Cu
- moved LED1 101.8 mm to (156.7, 66.9)
- moved R17 99.9 mm to (145.9, 77.2)
- moved R18 99.9 mm to (145.9, 79.0)
- moved Q1 95.1 mm to (170.1, 78.7), turned to 90 degrees
- moved R15 90.0 mm to (155.7, 71.7), turned to 90 degrees
- moved R14 89.9 mm to (156.5, 71.7), turned to 90 degrees
- moved R9 85.6 mm to (155.2, 66.9), turned to 90 degrees
- moved R10 84.2 mm to (156.6, 68.2), turned to 180 degrees
- moved R11 81.7 mm to (158.6, 67.6), turned to 90 degrees
- moved R3 78.7 mm to (163.4, 80.0), turned to 90 degrees
- moved U4 76.0 mm to (156.2, 74.2)
- moved R8 75.7 mm to (171.2, 78.7), turned to -90 degrees
- moved R1 69.7 mm to (173.1, 75.7)
- moved U7 67.2 mm to (169.9, 72.8), turned to 180 degrees
- moved C17 67.0 mm to (162.8, 69.1), turned to 180 degrees
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Routing:
- net Net-(D1-K): track 3.72 -> 0.00 mm
- net Net-(AN1-S): track 0.00 -> 2.83 mm
- net Net-(U3-ANT): track 0.00 -> 2.57 mm
- net Net-(AN1-Pad3): track 0.00 -> 1.59 mm
Other:
- board size 33.5 x 22.6 mm -> 29.2 x 22.6 mm
